Commit message: finished settings

File: stochlite_champ/stochlite_description/urdf/stochlite.urdf (robot description, URDF)
Before this commit: robot stochlite, 24 links, 23 joints
Links:
- link bl_toe_link: mass None -> 0.001; geometry collision sphere radius=0.014; visual sphere radius=0.0132
- link br_toe_link: mass None -> 0.001; geometry collision sphere radius=0.014; visual sphere radius=0.0132
- link fl_toe_link: mass None -> 0.001; geometry collision sphere radius=0.014; visual sphere radius=0.0132
- link fr_toe_link: mass None -> 0.001; geometry collision sphere radius=0.014; visual sphere radius=0.0132
